File: untitled.brd (EAGLE design)
At the start: 36 x 36 mm, 11 parts, among them IC1 ATTINY13-20PU, SW1 1825910-6

Commit message: Update untitled.brd
Parts:
- moved S2 5.57 mm to (87.0, 69.5)
- moved LED6 2.18 mm to (94.5, 70.5)
- moved LED1 1.85 mm to (99.6, 67.8)
- moved LED2 1.61 mm to (94.2, 50.3)
- moved LED3 1.30 mm to (99.7, 53.6)
- moved LED4 1.14 mm to (102.6, 60.8)
Routing:
- net N$1: track 12.9 -> 15.2 mm
- net N$2: track 18.2 -> 20.2 mm
- net VCC: track 35.3 -> 37.2 mm
- net N$3: track 16.8 -> 18.6 mm
- net N$4: track 13.1 -> 14.3 mm
- net N$6: track 35.6 -> 34.7 mm
- net N$5: track 12.6 -> 13.4 mm
Other:
- board size 36 x 36 mm -> 34.6 x 34.6 mm

Commit message: errors fixed
Parts:
- moved LED6 2.84 mm to (95.0, 73.3)
- moved LED3 2.34 mm to (101.5, 52.1)
- moved LED2 2.05 mm to (94.5, 48.3)
- moved S2 1.52 mm to (87.0, 67.9)
- moved LED1 1.48 mm to (100.8, 68.6)
- moved R9 0.80 mm to (102.5, 56.4)
- moved SW1 0.80 mm to (94.7, 60.1)
- moved LED4 0.76 mm to (102.6, 60.1)
- moved R1 0.51 mm to (101.7, 64.1)
Routing:
- net N$1: track 15.2 -> 20.4 mm
- net N$6: track 34.7 -> 38.6 mm
- net N$4: track 14.3 -> 17.0 mm
- net N$2: track 20.2 -> 22.1 mm
- net N$8: track 2.43 -> 1.26 mm
- net N$7: track 14.4 -> 15.1 mm
- net N$3: track 18.6 -> 19.1 mm
- net VCC: track 37.2 -> 36.7 mm
